File: Solder.kicad_pcb (KiCad board)
At the start: 2 copper layers, 41 x 28.5 mm, 5 parts

Commit message: Fixed mistake in wiring
Routing:
- net Net-(BT1--): track 17.7 -> 36.3 mm
Changed lines of the file:
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@@
+	)
+	(segment
+		(start 137.608075 101.81)
+		(end 143.6 95.818075)
+		(width 0.2)
+		(layer "F.Cu")
+		(net 1)
 	)
 	(segment
@@
 		(width 0.2)
 		(layer "F.Cu")
+		(net 1)
+	)
+	(segment
+		(start 127.5 101.81)
+		(end 137.608075 101.81)
+		(width 0.2)
+		(layer "F.Cu")
